Commit message: added robot dummy to the simulation

File: eurobot_sim/models/field.urdf (robot description, URDF)
Before this commit: robot field, 2 links, 1 joints
Links:
- added link main_robot; collision box size=0.4 0.2 0.34; visual box size=0.4 0.2 0.34
Joints:
- added joint table_to_main_robot: type floating, parent table, child main_robot

Commit message: fixed sizes/position of robot in the simulation

File: eurobot_sim/models/field.urdf (robot description, URDF)
Before this commit: robot field, 3 links, 2 joints
Links:
- link main_robot: geometry collision box size=0.42 0.19 0.35; visual box size=0.42 0.19 0.35

Commit message: added robot movement to the simulation

File: eurobot_sim/models/field.urdf (robot description, URDF)
Before this commit: robot field, 3 links, 2 joints
Links:
- removed link main_robot
Joints:
- removed joint table_to_main_robot

File: eurobot_sim/models/main_robot_by_stm.urdf (robot description, URDF)
Before this commit: robot main_robot, 1 links, 0 joints
Links:
- removed link main_robot
- added link main_robot_stm; collision box size=0.42 0.19 0.34; visual box size=0.42 0.19 0.34

Commit message: added table to the simulation

File: eurobot_sim/models/field.urdf (robot description, URDF)
Before this commit: robot field, 2 links, 1 joints
Links:
- link beacons: geometry collision cylinder length=0.1 radius=0.04; collision cylinder length=0.1 radius=0.04
- link table: mass None -> 165.19; geometry visual mesh filename=package://eurobot_sim/models/table.STL
