Commit message: some work on PF

File: eurobot_sim/models/main_robot_kf.urdf (robot description, URDF)
Before this commit: robot main_robot, 1 links, 0 joints
Links:
- removed link main_robot
- added link main_robot_kf; collision box size=0.42 0.19 0.34; visual box size=0.42 0.19 0.34

File: eurobot_sim/models/main_robot_pf.urdf (robot description, URDF)
Before this commit: robot main_robot_stm, 1 links, 0 joints
Links:
- removed link main_robot_stm
- added link main_robot_pf; collision box size=0.42 0.19 0.34; visual box size=0.42 0.19 0.34

File: eurobot_sim/models/main_robot_stm.urdf (robot description, URDF)
Before this commit: robot main_robot, 1 links, 0 joints
Links:
- removed link main_robot
- added link main_robot_stm; collision box size=0.42 0.19 0.34; visual box size=0.42 0.19 0.34
