Commit message: path planning from ROS navigation stack (local planning requires tuning)

File: eurobot_sim/models/main_robot_stm.urdf (robot description, URDF)
Before this commit: robot main_robot_stm, 1 links, 0 joints
Links:
- link main_robot_stm: geometry collision box size=0.1 0.19 0.34; collision box size=0.11 0.19 0.34
